File: A1200KB.kicad_pcb (KiCad board)
At the start: 2 copper layers, 450 x 125 mm, 101 parts, among them J1 Conn_01x32_Female, K1 ESC, K10 F9, K11 F10, K12 TILDE, K13 1, K14 2, K15 3, K16 4, K17 5, K18 6, K19 7, K2 F1, K20 8, K21 9, K22 0, K23 MINUS, K24 PLUS, K25 PIPE, K26 BS, K27 DEL, K28 HELP, K29 NUM_(, K3 F2, K30 NUM_), K31 NUM_DIV, K32 NUM_MULT, K33 TAB, K34 Q, K35 W, K36 E, K37 R, K38 T, K39 Y, K4 F3, K40 U, K41 I, K42 O, K43 P, K44 L.CURLY, K45 R.CURLY, K46 RETURN, K47 NUM_7, K48 NUM_8, K49 NUM_9, K5 F4, K50 NUM_MINUS, K51 CTRL, K52 CAPSLOCK, K53 A, K54 S, K55 D, K56 F, K57 G, K58 H, K59 J, K6 F5, K60 K, K61 L, K62 COLON, K63 ", K64 R.BLANK, K65 UP, K66 NUM_4, K67 NUM_5, K68 NUM_6, K69 NUM_PLUS, K7 F6, K70 L.SHIFT, K71 L.BLANK, K72 Z, K73 X, K74 C, K75 V, K76 B, K77 N, K78 M, K79 R.CROC, K8 F7, K80 L.CROC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

Commit message: Alps
Alps
Parts:
- removed the REF** at (198.2, 190.4)
- added G***: LOGO, Plate:plate 2000, F.Cu at (275.0, 138.0)
- added G***: LOGO, Alectardy98:Alectardy98 (3) Silk, F.Cu at (368.7, 186.2)
- added K100: R.CROC, Switch_Alps_Only:BIG_ALPS-1U, F.Cu at (451.3, 190.4)
- added K101: RETURN, Switch_Alps_Only:BIG_ALPS-1U, F.Cu at (329.9, 142.8)
- added K97: SPACE, Switch_Alps_Only:Big_ALPS-6.5U, F.Cu at (203.6, 190.4)
- added K98: SPACE, Switch_Alps_Only:BIG_ALPS-2.5U, F.Cu at (289.3, 190.4)
- added K99: PLUS, Switch_Alps_Only:BIG_ALPS-1U, F.Cu at (489.4, 171.3)
- K1, K13, K14, K15, K16, K17, K18, K19, K20, K21, K22, K23, K24, K25, K29, K30, K31, K32, K34, K35, K36, K37, K38, K39, K40, K41, K42, K43, K44, K45, K47, K48, K49, K50, K53, K54, K55, K56, K57, K58, K59, K60, K61, K62, K63, K64, K65, K66, K67, K68, K69, K71, K72, K73, K74, K75, K76, K77, K78, K79, K80, K81, K83, K84, K85, K86, K87, K88, K96: footprint MX_Alps_Hybrid:MXOnly-1U-NoLED -> Switch_Alps_Only:BIG_ALPS-1U
- K10, K11, K2, K3, K4, K5, K6, K7, K8, K9: footprint MX_Alps_Hybrid:MXOnly-1.25U-NoLED -> Switch_Alps_Only:BIG_ALPS-1.25U
- K12: footprint MX_Alps_Hybrid:MXOnly-1.5U-NoLED -> Switch_Alps_Only:BIG_ALPS-1.25U
- K26: footprint MX_Alps_Hybrid:MXOnly-1U-NoLED -> Switch_Alps_Only:BIG_ALPS-1.25U
- K27, K28: footprint MX_Alps_Hybrid:MXOnly-1.5U-NoLED -> Switch_Alps_Only:BIG_ALPS-1U
- K33: footprint MX_Alps_Hybrid:MXOnly-2U-NoLED -> Switch_Alps_Only:BIG_ALPS-1.75U
- K46: footprint MX_Alps_Hybrid:MXOnly-ISO -> Switch_Alps_Only:BIG_ALPS-1U
- K51, K90, K91, K94: footprint MX_Alps_Hybrid:MXOnly-1.25U-NoLED -> Switch_Alps_Only:BIG_ALPS-1U
- K52: footprint MX_Alps_Hybrid:MXOnly-1U -> Switch_Alps_Only:BIG_ALPS-1U
- K70: footprint MX_Alps_Hybrid:MXOnly-1.75U-NoLED -> Switch_Alps_Only:BIG_ALPS-2.5U
- K82: footprint MX_Alps_Hybrid:MXOnly-2.75U-NoLED -> Switch_Alps_Only:BIG_ALPS-2U
- K89, K95: footprint MX_Alps_Hybrid:MXOnly-2U-NoLED -> Switch_Alps_Only:BIG_ALPS-1U
- K92: footprint MX_Alps_Hybrid:MXOnly-7U-NoLED -> Switch_Alps_Only:BIG_ALPS-2U
- K93: value R.AMIGA -> DEL; footprint MX_Alps_Hybrid:MXOnly-1.25U-NoLED -> Switch_Alps_Only:BIG_ALPS-1U
- moved K71 204.7 mm to (298.9, 171.3)
- moved K93 131.8 mm to (403.6, 114.2)
- moved K92 75.6 mm to (122.6, 190.4), turned to 0 degrees
- moved K28 13.6 mm to (384.6, 114.2)
- moved K89 9.62 mm to (489.4, 190.4), turned to 0 degrees
- moved K95 9.00 mm to (432.2, 190.4), turned to 0 degrees
- moved K70 7.05 mm to (75.0, 171.3)
- moved K82 6.99 mm to (327.4, 171.3)
- moved K91 6.67 mm to (94.1, 190.4)
- moved K74 4.83 mm to (146.5, 171.3)
- moved K72 4.83 mm to (108.4, 171.3)
- moved K73 4.83 mm to (127.4, 171.3)
- moved K75 4.83 mm to (165.5, 171.3)
- moved K76 4.83 mm to (184.6, 171.3)
- moved K77 4.83 mm to (203.6, 171.3)
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Connections:
- J1 pad 32: Net-(J1-Pad32) -> unconnected-(J1-Pin_32-Pad32)
- K93 pad 1: /30 -> /28
- K93 pad 2: /10 -> /2
Routing:
- net /15: track 551.7 -> 1010.8 mm, vias 2 -> 1
- net /24: track 421.4 -> 707.3 mm
- net /31: track 243.0 -> 0.00 mm, vias 2 -> 0
- net /27: track 449.1 -> 684.9 mm, vias 3 -> 1
- net /3: track 493.1 -> 723.4 mm, vias 2 -> 1
- net /9: track 198.2 -> 0.00 mm, vias 1 -> 0
- net /10: track 173.9 -> 0.00 mm, vias 1 -> 0
- net /18: track 483.4 -> 656.3 mm, vias 3 -> 2
- net /17: track 514.7 -> 678.0 mm, vias 3 -> 0
- net /1: track 384.6 -> 526.3 mm, vias 2 -> 0
- net /2: track 427.2 -> 541.8 mm, vias 2 -> 0
- net /5: track 405.5 -> 502.8 mm, vias 3 -> 0
- net /16: track 538.7 -> 603.4 mm, vias 4 -> 1
- net /25: track 301.4 -> 355.8 mm, vias 2 -> 1
- net /7: track 454.3 -> 505.1 mm, vias 1 -> 0
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Other:
- net class Default removed
- board text added: "Dec. 2023"
- board text added: "Rev. Alps"
- board text removed: "+"
- board text removed: "7,103"
- board text removed: "7,38"
- board text removed: "7,7"
- board text removed: "July 2021"
- board text removed: "Rev.4"
